Commit message: Functioning restructured motors and CRSF

File: ardagv/urdf/ardagv_model.urdf.xacro (robot description, xacro)
@@ -2,6 +2,6 @@
 <robot xmlns:xacro="http://www.ros.org/wiki/xacro">
 <xacro:macro name="ardagv_model" params="name">
-	<link name="${name}_base_link"></link> <!-- ground-level, below centerpoint between wheels -->
-	<link name="${name}_chasis">
+	<link name="base_link"></link>
+	<link name="chasis">
 		<visual>
 			<origin xyz="0 0 0.08" rpy="0 0 0" />
@@ -14,9 +14,9 @@
 		</material>
 	</link>
-	<joint name="${name}_base_to_chasis" type="fixed">
-		<parent link="${name}_base_link" />
-		<child link="${name}_chasis" />
+	<joint name="base_to_chasis" type="fixed">
+		<parent link="base_link" />
+		<child link="chasis" />
 	</joint>
-	<link name="${name}_wheel_left">
+	<link name="wheel_left">
 		<visual>
 			<geometry>
@@ -28,7 +28,7 @@
 		</material>
 	</link>
-	<joint name="${name}_motor_left" type="continuous">
-		<parent link="${name}_base_link" />
-		<child link="${name}_wheel_left" />
+	<joint name="motor_left" type="continuous">
+		<parent link="base_link" />
+		<child link="wheel_left" />
 		<origin xyz="0 0.01225 0.05" rpy="1.570796326794897 0 0" />
 		<command_interface name="velocity"> <!-- RPM limits: -->
@@ -37,5 +37,5 @@
 		</command_interface>
 	</joint>
-	<link name="${name}_wheel_right">
+	<link name="wheel_right">
 		<visual>
 			<geometry>
@@ -47,7 +47,7 @@
 		</material>
 	</link>
-	<joint name="${name}_motor_right" type="continuous">
-		<parent link="${name}_base_link" />
-		<child link="${name}_wheel_right" />
+	<joint name="motor_right" type="continuous">
+		<parent link="base_link" />
+		<child link="wheel_right" />
 		<origin xyz="0 -0.01225 0.05" rpy="-1.570796326794897 0 0" />
 		<command_interface name="velocity"> <!-- RPM limits: -->
@@ -56,6 +56,6 @@
 		</command_interface>
 	</joint>
-	<sensor name="${name}_tof">
-		<parent link="${name}_base_link" />
+	<sensor name="tof">
+		<parent link="base_link" />
 		<origin xyz="0.3 0 0.05" rpy="0 0 0" /> <!-- TODO: orientation -->
 		<camera>
@@ -64,6 +64,6 @@
 		</camera>
 	</sensor>
-	<sensor name="${name}_imu">
-		<parent link="${name}_base_link" />
+	<sensor name="imu">
+		<parent link="base_link" />
 		<origin xyz="0.133 -0.01 0.05" rpy="0 0 0" /> <!-- TODO: orientation -->
 	</sensor>

File: ardagv/urdf/ardagv_ros2_control.urdf.xacro (robot description, xacro)
@@ -10,13 +10,13 @@
     <param name="master_bin"></param>
   </hardware>
-  <joint name="${name}_motor_left"> <!-- must correspond to joint defined in ardagv_model.urdf -->
+  <joint name="motor_left"> <!-- must correspond to joint defined in ardagv_model.urdf -->
     <command_interface name="velocity"/>
-    <param name="device_name">${name}_motor_left</param> <!-- must correspond to node name which controls this joint -->
+    <param name="device_name">drive_left</param> <!-- must correspond to node name which controls this joint -->
     <state_interface name="position"/>
     <state_interface name="velocity"/>
   </joint>
-  <joint name="${name}_motor_right">
+  <joint name="motor_right">
     <command_interface name="velocity"/>
-    <param name="device_name">${name}_motor_right</param>
+    <param name="device_name">drive_right</param>
     <state_interface name="position"/>
     <state_interface name="velocity"/>

Commit message: Corrected URDF model

File: ardagv/urdf/ardagv_model.urdf.xacro (robot description, xacro)
@@ -2,157 +2,72 @@
 <robot xmlns:xacro="http://www.ros.org/wiki/xacro">
 <xacro:macro name="ardagv_model" params="name">
-	<link name="base_link"></link>
-	<link name="chasis">
-		<visual>
-			<origin xyz="0 0 0.08" rpy="0 0 0" />
-			<geometry>
-				<box size="0.6 0.3 0.15" />
-			</geometry>
-		</visual>
-		<material name="chasis-material">
-			<color rgba="0.5 0.5 0.5 1" />
-		</material>
-	</link>
-	<joint name="base_to_chasis" type="fixed">
-		<parent link="base_link" />
-		<child link="chasis" />
-	</joint>
-	<link name="wheel_left">
-		<visual>
-			<geometry>
-				<cylinder radius="0.05" length="0.025" />
-			</geometry>
-		</visual>
-		<material name="wheel-material">
-			<color rgba="0.2 0.2 0.2 1" />
-		</material>
-	</link>
-	<joint name="motor_left" type="continuous">
-		<parent link="base_link" />
-		<child link="wheel_left" />
-		<origin xyz="0 0.01225 0.05" rpy="1.570796326794897 0 0" />
-		<command_interface name="velocity"> <!-- RPM limits: -->
-			<param name="min">-18</param>
-			<param name="max">18</param>
-		</command_interface>
-	</joint>
-	<link name="wheel_right">
-		<visual>
-			<geometry>
-				<cylinder radius="0.05" length="0.025" />
-			</geometry>
-		</visual>
-		<material name="wheel-material">
-			<color rgba="0.2 0.2 0.2 1" />
-		</material>
-	</link>
-	<joint name="motor_right" type="continuous">
-		<parent link="base_link" />
-		<child link="wheel_right" />
-		<origin xyz="0 -0.01225 0.05" rpy="-1.570796326794897 0 0" />
-		<command_interface name="velocity"> <!-- RPM limits: -->
-			<param name="min">-18</param>
-			<param name="max">18</param>
-		</command_interface>
-	</joint>
-	<sensor name="tof">
-		<parent link="base_link" />
-		<origin xyz="0.3 0 0.05" rpy="0 0 0" /> <!-- TODO: orientation -->
-		<camera>
-			<image width="512" height="512" hfov="2" format="mono16" near="0.4" far="5" /> <!-- TODO: change FOV, radians -->
-			<image width="512" height="512" hfov="2" format="mono16" near="0.4" far="5" />
-		</camera>
-	</sensor>
-	<sensor name="imu">
-		<parent link="base_link" />
-		<origin xyz="0.133 -0.01 0.05" rpy="0 0 0" /> <!-- TODO: orientation -->
-	</sensor>
-	<!-- OLD:
-	<link name="${name}_world"></link>
-  <link name="${name}_base_link">
-    <visual>
-      <origin xyz="0 0 0" rpy="0 0 0" />
-      <geometry>
-        <box size="0.5 0.3 0.2" />
-      </geometry>
-      <material name="base_link-material">
-        <color rgba="0.5271151256969157 0.5271151256969157 0.5271151256969157 1" />
-      </material>
-    </visual>
-    <collision>
-      <origin xyz="0 0 0" rpy="0 0 0" />
-      <geometry>
-        <box size="0.5 0.3 0.2" />
-      </geometry>
-    </collision>
-    <inertial>
-      <origin xyz="0 0 0" rpy="0 0 0" />
-      <mass value="1" />
-      <inertia ixx="0.16666666666666666" ixy="0" ixz="0" iyy="0.16666666666666666" iyz="0" izz="0.16666666666666666" />
-    </inertial>
-  </link>
-  <joint name="${name}_wheel_left" type="continuous">
-	  <parent link="${name}_base_link" />
-	  <child link="${name}_left_wheel" />
-    <origin xyz="0 0.16 -0.05" rpy="1.570796326794897 0 0" />
-    <command_interface name="velocity">
-      <param name="min">-18</param>
-      <param name="max">18</param>
-    </command_interface>
-  </joint>
-  <link name="${name}_left_wheel">
-    <visual>
-      <origin xyz="0 0 0" rpy="0 0 0" />
-      <geometry>
-        <cylinder radius="0.05" length="0.01" />
-      </geometry>
-      <material name="left_wheel-material">
-        <color rgba="0.21223075740342198 0.21586050010324417 0.41254261347374327 1" />
-      </material>
-    </visual>
-    <collision>
-      <origin xyz="0 0 0" rpy="0 0 0" />
-      <geometry>
-        <cylinder radius="0.05" length="0.01" />
-      </geometry>
-    </collision>
-    <inertial>
-      <origin xyz="0 0 0" rpy="0 0 0" />
-      <mass value="1" />
-      <inertia ixx="0.3333333333333333" ixy="0" ixz="0" iyy="0.5" iyz="0" izz="0.3333333333333333" />
-    </inertial>
-  </link>
-  <joint name="${name}_wheel_right" type="continuous">
-	  <parent link="${name}_base_link" />
-	  <child link="${name}_right_wheel" />
-    <origin xyz="0 -0.16 -0.05" rpy="1.570796326794897 0 0" />
-    <command_interface name="velocity">
-      <param name="min">-18</param>
-      <param name="max">18</param>
-    </command_interface>
-  </joint>
-  <link name="${name}_right_wheel">
-    <visual>
-      <origin xyz="0 0 0" rpy="0 0 0" />
-      <geometry>
-        <cylinder radius="0.05" length="0.01" />
-      </geometry>
-      <material name="right_wheel-material">
-        <color rgba="0.21223075740342198 0.21586050010324417 0.41254261347374327 1" />
-      </material>
-    </visual>
-    <collision>
-      <origin xyz="0 0 0" rpy="0 0 0" />
-      <geometry>
-        <cylinder radius="0.05" length="0.01" />
-      </geometry>
-    </collision>
-    <inertial>
-      <origin xyz="0 0 0" rpy="0 0 0" />
-      <mass value="1" />
-      <inertia ixx="0.3333333333333333" ixy="0" ixz="0" iyy="0.5" iyz="0" izz="0.3333333333333333" />
-    </inertial>
-  </link>
-	-->
+        <link name="base_link"></link>
+        <link name="chasis">
+                <visual>
+                        <origin xyz="0 0 0.08" rpy="0 0 0" />
+                        <geometry>
+                                <box size="0.6 0.3 0.15" />
+                        </geometry>
+                        <material name="chasis-material">
+                                <color rgba="0.5 0.5 0.5 1" />
+                        </material>
+                </visual>
+        </link>
+        <joint name="base_to_chasis" type="fixed">
+                <parent link="base_link" />
+                <child link="chasis" />
+        </joint>
+        <link name="wheel_left">
+                <visual>
+                        <origin xyz="0 0 0" rpy="0 0 0" />
+                        <geometry>
+                                <cylinder radius="0.05" length="0.025" />
+                        </geometry>
+                        <material name="wheel-material">
+                                <color rgba="0.2 0.2 0.2 1" />
+                        </material>
+                </visual>
+        </link>
+        <joint name="motor_left" type="continuous">
+                <parent link="base_link" />
+                <child link="wheel_left" />
+                <origin xyz="0 0.1225 0.05" rpy="1.5708 0 0" />
+                <command_interface name="velocity"> <!-- RPM limits: -->
+                        <param name="min">-18</param>
+                        <param name="max">18</param>
+                </command_interface>
+        </joint>
+        <link name="wheel_right">
+                <visual>
+                        <origin xyz="0 0 0" rpy="0 0 0" />
+                        <geometry>
+                                <cylinder radius="0.05" length="0.025" />
+                        </geometry>
+                        <material name="wheel-material">
+                                <color rgba="0.2 0.2 0.2 1" />
+                        </material>
+                </visual>
+        </link>
+        <joint name="motor_right" type="continuous">
+                <parent link="base_link" />
+                <child link="wheel_right" />
+                <origin xyz="0 -0.1225 0.05" rpy="-1.5708 0 0" />
+                <command_interface name="velocity"> <!-- RPM limits: -->
+                        <param name="min">-18</param>
+                        <param name="max">18</param>
+                </command_interface>
+        </joint>
+        <sensor name="tof">
+                <parent link="base_link" />
+                <origin xyz="0.3 0 0.05" rpy="0 0 0" /> <!-- TODO: orientation -->
+                <camera>
+                        <image width="512" height="512" hfov="2" format="mono16" near="0.4" far="5" /> <!-- TODO: change FOV, radians -->
+                        <image width="512" height="512" hfov="2" format="mono16" near="0.4" far="5" />
+                </camera>
+        </sensor>
+        <sensor name="imu">
+                <parent link="base_link" />
+                <origin xyz="0.133 -0.01 0.05" rpy="0 0 0" /> <!-- TODO: orientation -->
+        </sensor>
 </xacro:macro>
 </robot>

Commit message: Add TOF and IMU frames, tweak CRSF node
Signed-off-by: Ioan Dragomir <ioan.dragomir@analog.com>

File: ardagv/urdf/ardagv_model.urdf.xacro (robot description, xacro)
@@ -58,4 +58,18 @@
                 </command_interface>
         </joint>
+	<link name="cam1_adtf31xx_optical">
+	</link>
+	<joint name="tof_position" type="fixed">
+		<parent link="base_link" />
+                <child link="cam1_adtf31xx_optical" />
+		<origin xyz="0.3 0 0.05" rpy="1.5708 0 1.5708" />
+	</joint>
+	<link name="imu">
+	</link>
+	<joint name="imu_position" type="fixed">
+		<parent link="base_link" />
+                <child link="imu" />
+		<origin xyz="0.133 -0.01 0.05" rpy="1.5708 0 0" />
+	</joint>
         <sensor name="tof">
                 <parent link="base_link" />

Commit message: urdf: Add cam1_laser link, replace tof _optical

File: ardagv/urdf/ardagv_model.urdf.xacro (robot description, xacro)
@@ -58,18 +58,27 @@
                 </command_interface>
         </joint>
-	<link name="cam1_adtf31xx_optical">
-	</link>
-	<joint name="tof_position" type="fixed">
-		<parent link="base_link" />
-                <child link="cam1_adtf31xx_optical" />
-		<origin xyz="0.3 0 0.05" rpy="1.5708 0 1.5708" />
-	</joint>
-	<link name="imu">
-	</link>
-	<joint name="imu_position" type="fixed">
-		<parent link="base_link" />
+        <link name="cam1_adtf31xx">
+        </link>
+        <joint name="tof_position" type="fixed">
+                <parent link="base_link" />
+                <!--<child link="cam1_adtf31xx_optical" />
+                <origin xyz="0.3 0 0.05" rpy="1.5708 0 1.5708" />-->
+                <child link="cam1_adtf31xx" />
+                <origin xyz="0.3 0 0.05" rpy="0 0 0" />
+        </joint>
+        <link name="cam1_laser">
+        </link>
+        <joint name="laser_position" type="fixed">
+                <parent link="base_link" />
+                <child link="cam1_laser" />
+                <origin xyz="0.3 0 0.05" rpy="0 0 0" />
+        </joint>
+        <link name="imu">
+        </link>
+        <joint name="imu_position" type="fixed">
+                <parent link="base_link" />
                 <child link="imu" />
-		<origin xyz="0.133 -0.01 0.05" rpy="1.5708 0 0" />
-	</joint>
+                <origin xyz="0.133 -0.01 0.05" rpy="1.5708 0 0" />
+        </joint>
         <sensor name="tof">
                 <parent link="base_link" />
