Commit message: ardagv: Add simulator to main robot script

File: ardagv/urdf/ardagv_all.urdf.xacro (robot description, xacro)
@@ -1,10 +1,10 @@
 <?xml version="1.0"?>
 <robot xmlns:xacro="http://www.ros.org/wiki/xacro" name="ardagv">
-	<xacro:arg name="name" default="ardagv" /> <!-- prefix for all URDF names -->
-	<xacro:arg name="config_dir" default="$(find ardagv)/config/" /> <!-- Install directory containing CANopen config, .dcf files -->
-	<xacro:arg name="can_iface" default="can1" />
-	<xacro:include filename="$(find ardagv)/urdf/ardagv_ros2_control.urdf.xacro" />
-	<xacro:include filename="$(find ardagv)/urdf/ardagv_model.urdf.xacro" />
-	<xacro:ardagv_ros2_control name="$(arg name)" config_dir="$(arg config_dir)" can_iface="$(arg can_iface)" />
-	<xacro:ardagv_model name="$(arg name)" />
+	<xacro:arg name="sim_mode" default="false"/> <!-- true if running in simulation -->
+	<xacro:include filename="ardagv_ros2_control.urdf.xacro"/>
+	<xacro:include filename="ardagv_model.urdf.xacro"/>
+	<xacro:include filename="lidar.xacro" />
+	<xacro:include filename="imu.xacro" />
+	<xacro:include filename="camera.xacro" />
+	<!-- <xacro:include filename="depth_camera.xacro" /> -->
 </robot>

File: ardagv/urdf/ardagv_model.urdf.xacro (robot description, xacro)
@@ -1,96 +1,145 @@
 <?xml version="1.0"?>
-<robot xmlns:xacro="http://www.ros.org/wiki/xacro">
-<xacro:macro name="ardagv_model" params="name">
-        <link name="base_link"></link>
-        <link name="chasis">
-                <visual>
-                        <origin xyz="0 0 0.08" rpy="0 0 0" />
-                        <geometry>
-                                <box size="0.6 0.3 0.15" />
-                        </geometry>
-                        <material name="chasis-material">
-                                <color rgba="0.5 0.5 0.5 1" />
-                        </material>
-                </visual>
+<robot xmlns:xacro="http://www.ros.org/wiki/xacro" >
+    <xacro:include filename="inertial_macros.xacro"/>
+    <xacro:property name="chassis_length" value="0.60"/>
+    <xacro:property name="chassis_width" value="0.30"/>
+    <xacro:property name="chassis_height" value="0.15"/>
+    <xacro:property name="base_width" value="0.22"/>
+    <xacro:property name="chassis_zoff" value="0.08"/>
+    <xacro:property name="chassis_mass" value="1.0"/>
+    <xacro:property name="wheel_radius" value="0.05"/>
+    <xacro:property name="wheel_width" value="0.025"/>
+    <xacro:property name="wheel_mass" value="0.05"/>
+    <xacro:property name="caster_wheel_radius" value="0.025"/>
+    <xacro:property name="caster_wheel_mass" value="0.01"/>
+    <xacro:property name="caster_wheel_zoff" value="${caster_wheel_radius}"/>
+    <material name="cyan"><color rgba="0 1.0 1.0 1.0"/></material>
+    <material name="gray"><color rgba="0.5 0.5 0.5 1.0"/></material>
+    <material name="white"><color rgba="1 1 1 1"/></material>
+    <material name="orange"><color rgba="1 0.3 0.1 1"/></material>
+    <material name="blue"><color rgba="0.2 0.2 1 1"/></material>
+    <material name="black"><color rgba="0 0 0 1"/></material>
+    <material name="red"><color rgba="1 0 0 1"/></material>
+    <!-- BASE LINK -->
+    <link name="base_link"></link>
+    <!-- BASE_FOOTPRINT LINK -->
+    <joint name="base_footprint_joint" type="fixed">
+        <parent link="base_link"/>
+        <child link="base_footprint"/>
+        <origin xyz="0 0 0" rpy="0 0 0"/>
+    </joint>
+    <link name="base_footprint"></link>
+    <!-- CHASSIS LINK -->
+    <joint name="chassis_joint" type="fixed">
+        <parent link="base_link"/>
+        <child link="chassis"/>
+        <origin xyz="0 0 ${chassis_zoff}"/>
+    </joint>
+    <link name="chassis">
+        <visual>
+            <origin xyz="0 0 ${chassis_zoff}"/>
+            <geometry>
+                <box size="${chassis_length} ${chassis_width} ${chassis_height}"/>
+            </geometry>
+            <material name="cyan"/>
+        </visual>
+        <collision>
+            <origin xyz="0 0 ${chassis_zoff}"/>
+            <geometry>
+                <box size="${chassis_length} ${chassis_width} ${chassis_height}"/>
+            </geometry>
+        </collision>
+        <xacro:inertial_box mass="0.5" x="${chassis_length}" y="${chassis_width}" z="${chassis_height}">
+            <origin xyz="0 0 ${chassis_zoff}" rpy="0 0 0"/>
+        </xacro:inertial_box>
+    </link>
+    <gazebo reference="chassis">
+        <material>Gazebo/Gray</material>
+    </gazebo>
+    <!-- LEFT WHEEL LINK -->
+    <joint name="left_wheel_joint" type="continuous">
+        <parent link="base_link"/>
+        <child link="left_wheel"/>
+        <origin xyz="0 ${(base_width + wheel_width)/2} ${wheel_radius}" rpy="-${pi/2} 0 0" />
+        <axis xyz="0 0 1"/>
+    </joint>
+    <link name="left_wheel">
+        <visual>
+            <geometry>
+                <cylinder radius="${wheel_radius}" length="${wheel_width}"/>
+            </geometry>
+            <material name="blue"/>
+        </visual>
+        <collision>
+            <geometry>
+                <sphere radius="${wheel_radius}"/>
+            </geometry>
+        </collision>
+        <xacro:inertial_cylinder mass="${wheel_mass}" length="${wheel_width}" radius="${wheel_radius}">
+            <origin xyz="0 0 0" rpy="0 0 0"/>
+        </xacro:inertial_cylinder>
+    </link>
+    <gazebo reference="left_wheel">
+        <material>Gazebo/Blue</material>
+    </gazebo>
+    <!-- RIGHT WHEEL LINK -->
+    <joint name="right_wheel_joint" type="continuous">
+        <parent link="base_link"/>
+        <child link="right_wheel"/>
+        <origin xyz="0 ${-(base_width + wheel_width)/2} ${wheel_radius}" rpy="${pi/2} 0 0" />
+        <axis xyz="0 0 -1"/>
+    </joint>
+    <link name="right_wheel">
+        <visual>
+            <geometry>
+                <cylinder radius="${wheel_radius}" length="${wheel_width}"/>
+            </geometry>
+            <material name="blue"/>
+        </visual>
+        <collision>
+            <geometry>
+                <sphere radius="${wheel_radius}"/>
+            </geometry>
+        </collision>
+        <xacro:inertial_cylinder mass="${wheel_mass}" length="${wheel_width}" radius="${wheel_radius}">
+            <origin xyz="0 0 0" rpy="0 0 0"/>
+        </xacro:inertial_cylinder>
+    </link>
+    <gazebo reference="right_wheel">
+        <material>Gazebo/Blue</material>
+    </gazebo>
+    <!-- CASTER WHEEL LINKS -->
+    <xacro:macro name="caster_wheel" params="prefix x_reflect y_reflect">
+        <link name="${prefix}_link">
+            <visual>
+                <geometry>
+                    <sphere radius="${caster_wheel_radius}"/>
+                </geometry>
+                <material name="cyan"/>
+            </visual>
+            <collision>
+                <origin xyz="0 0 0" rpy="0 0 0"/>
+                <geometry>
+                    <sphere radius="${caster_wheel_radius}"/>
+                </geometry>
+            </collision>
+            <xacro:inertial_sphere mass="${caster_wheel_mass}" radius="${caster_wheel_radius}">
+                <origin xyz="0 0 0" rpy="0 0 0"/>
+            </xacro:inertial_sphere>
         </link>
-        <joint name="base_to_chasis" type="fixed">
-                <parent link="base_link" />
-                <child link="chasis" />
+        <joint name="${prefix}_joint" type="fixed">
+            <parent link="base_link"/>
+            <child link="${prefix}_link"/>
+            <origin xyz="${x_reflect*(chassis_length/2-caster_wheel_radius)} ${y_reflect*(base_width/2-caster_wheel_radius)} ${caster_wheel_zoff}" rpy="0 0 0"/>
         </joint>
-        <link name="wheel_left">
-                <visual>
-                        <origin xyz="0 0 0" rpy="0 0 0" />
-                        <geometry>
-                                <cylinder radius="0.05" length="0.025" />
-                        </geometry>
-                        <material name="wheel-material">
-                                <color rgba="0.2 0.2 0.2 1" />
-                        </material>
-                </visual>
-        </link>
-        <joint name="motor_left" type="continuous">
-                <parent link="base_link" />
-                <child link="wheel_left" />
-                <origin xyz="0 0.1225 0.05" rpy="1.5708 0 0" />
-                <command_interface name="velocity"> <!-- RPM limits: -->
-                        <param name="min">-18</param>
-                        <param name="max">18</param>
-                </command_interface>
-        </joint>
-        <link name="wheel_right">
-                <visual>
-                        <origin xyz="0 0 0" rpy="0 0 0" />
-                        <geometry>
-                                <cylinder radius="0.05" length="0.025" />
-                        </geometry>
-                        <material name="wheel-material">
-                                <color rgba="0.2 0.2 0.2 1" />
-                        </material>
-                </visual>
-        </link>
-        <joint name="motor_right" type="continuous">
-                <parent link="base_link" />
-                <child link="wheel_right" />
-                <origin xyz="0 -0.1225 0.05" rpy="-1.5708 0 0" />
-                <command_interface name="velocity"> <!-- RPM limits: -->
-                        <param name="min">-18</param>
-                        <param name="max">18</param>
-                </command_interface>
-        </joint>
-        <link name="cam1_adtf31xx">
-        </link>
-        <joint name="tof_position" type="fixed">
-                <parent link="base_link" />
-                <!--<child link="cam1_adtf31xx_optical" />
-                <origin xyz="0.3 0 0.05" rpy="1.5708 0 1.5708" />-->
-                <child link="cam1_adtf31xx" />
-                <origin xyz="0.3 0 0.05" rpy="0 0 0" />
-        </joint>
-        <link name="cam1_laser">
-        </link>
-        <joint name="laser_position" type="fixed">
-                <parent link="base_link" />
-                <child link="cam1_laser" />
-                <origin xyz="0.3 0 0.05" rpy="0 0 0" />
-        </joint>
-        <link name="imu">
-        </link>
-        <joint name="imu_position" type="fixed">
-                <parent link="base_link" />
-                <child link="imu" />
-                <origin xyz="0.133 -0.01 0.05" rpy="1.5708 0 0" />
-        </joint>
-        <sensor name="tof">
-                <parent link="base_link" />
-                <origin xyz="0.3 0 0.05" rpy="0 0 0" /> <!-- TODO: orientation -->
-                <camera>
-                        <image width="512" height="512" hfov="2" format="mono16" near="0.4" far="5" /> <!-- TODO: change FOV, radians -->
-                        <image width="512" height="512" hfov="2" format="mono16" near="0.4" far="5" />
-                </camera>
-        </sensor>
-        <sensor name="imu">
-                <parent link="base_link" />
-                <origin xyz="0.133 -0.01 0.05" rpy="0 0 0" /> <!-- TODO: orientation -->
-        </sensor>
-</xacro:macro>
+        <gazebo reference="${prefix}_link">
+            <material>Gazebo/Blue</material>
+            <mu1 value="0.001"/>
+            <mu2 value="0.001"/>
+        </gazebo>
+    </xacro:macro>
+    <xacro:caster_wheel prefix="front_left_caster" x_reflect="1" y_reflect="1"/>
+    <xacro:caster_wheel prefix="front_right_caster" x_reflect="1" y_reflect="-1"/>
+    <xacro:caster_wheel prefix="rear_left_caster" x_reflect="-1" y_reflect="1"/>
+    <xacro:caster_wheel prefix="rear_right_caster" x_reflect="-1" y_reflect="-1"/>
 </robot>

File: ardagv/urdf/ardagv_ros2_control.urdf.xacro (robot description, xacro)
@@ -1,35 +1,70 @@
 <?xml version="1.0"?>
 <robot xmlns:xacro="http://www.ros.org/wiki/xacro">
-<xacro:macro name="ardagv_ros2_control" params="name config_dir can_iface">
-<ros2_control name="${name}_control" type="system">
-	<!--<hardware>
-    <plugin>canopen_ros2_control/RobotSystem</plugin>
-    <param name="bus_config">${config_dir}/bus.yml</param>
-    <param name="master_config">${config_dir}/master.dcf</param>
-    <param name="can_interface_name">${can_iface}</param>
-    <param name="master_bin"></param>
-	</hardware>-->
-  <hardware>
-    <plugin>canopen_ros2_control/Cia402System</plugin>
-    <param name="bus_config">${config_dir}/bus.yml</param>
-    <param name="master_config">${config_dir}/master.dcf</param>
-    <param name="can_interface_name">${can_iface}</param>
-    <param name="master_bin"></param>
-  </hardware>
-  <joint name="motor_left"> <!-- must correspond to joint defined in ardagv_model.urdf -->
-    <command_interface name="velocity"/>
-    <param name="device_name">drive_left</param> <!-- must correspond to node name which controls this joint -->
-    <param name="node_id">22</param>
-    <state_interface name="position"/>
-    <state_interface name="velocity"/>
-  </joint>
-  <joint name="motor_right">
-    <command_interface name="velocity"/>
-    <param name="device_name">drive_right</param>
-    <param name="node_id">20</param>
-    <state_interface name="position"/>
-    <state_interface name="velocity"/>
-  </joint>
-</ros2_control>
-</xacro:macro>
+    <xacro:unless value="$(arg sim_mode)">
+        <ros2_control name="$ardagv_control" type="system">
+            <!--<hardware>
+                <plugin>canopen_ros2_control/RobotSystem</plugin>
+                <param name="bus_config">${config_dir}/bus.yml</param>
+                <param name="master_config">${config_dir}/master.dcf</param>
+                <param name="can_interface_name">${can_iface}</param>
+                <param name="master_bin"></param>
+            </hardware>-->
+            <hardware>
+                <plugin>canopen_ros2_control/Cia402System</plugin>
+                <param name="bus_config">$(find ardagv)/config/bus.yml</param>
+                <param name="master_config">$(find ardagv)/config/master.dcf</param>
+                <param name="can_interface_name">can1</param>
+                <param name="master_bin"></param>
+            </hardware>
+            <joint name="left_wheel_joint"> <!-- must correspond to joint defined in ardagv_model.urdf -->
+                <command_interface name="velocity">
+                    <param name="min">-18</param>
+                    <param name="max">18</param>
+                </command_interface>
+                <param name="device_name">drive_left</param> <!-- must correspond to node name which controls this joint -->
+                <param name="node_id">22</param>
+                <state_interface name="position"/>
+                <state_interface name="velocity"/>
+            </joint>
+            <joint name="right_wheel_joint">
+                <command_interface name="velocity">
+                    <param name="min">-18</param>
+                    <param name="max">18</param>
+                </command_interface>
+                <param name="device_name">drive_right</param>
+                <param name="node_id">20</param>
+                <state_interface name="position"/>
+                <state_interface name="velocity"/>
+            </joint>
+        </ros2_control>
+    </xacro:unless>
+    <xacro:if value="$(arg sim_mode)">
+        <ros2_control name="GazeboSystem" type="system">
+            <hardware>
+                <plugin>gazebo_ros2_control/GazeboSystem</plugin>
+            </hardware>
+            <joint name="left_wheel_joint">
+                <command_interface name="velocity">
+                    <param name="min">-18</param>
+                    <param name="max">18</param>
+                </command_interface>
+                <state_interface name="velocity"/>
+                <state_interface name="position"/>
+            </joint>
+            <joint name="right_wheel_joint">
+                <command_interface name="velocity">
+                    <param name="min">-18</param>
+                    <param name="max">18</param>
+                </command_interface>
+                <state_interface name="velocity"/>
+                <state_interface name="position"/>
+            </joint>
+        </ros2_control>
+    </xacro:if>
+    <gazebo>
+        <plugin name="gazebo_ros2_control" filename="libgazebo_ros2_control.so">
+            <parameters>$(find ardagv)/config/ros2_controllers.yaml</parameters>
+            <parameters>$(find ardagv)/config/gaz_ros2_ctl_use_sim.yaml</parameters>
+        </plugin>
+    </gazebo>
 </robot>
